Commit message: paper: NEW URDF 100% working

File: src/viz/models/orca_test/urdf/orca_test.urdf (robot description, URDF)
Before this commit: robot converted_robot, 39 links, 38 joints
Links:
- removed link AP-Assembly_0c2e1cd6
- removed link AP-Assembly_0c2e1cd6_joint_jointbody
- removed link AP-Assembly_22c0dde4
- removed link AP-Assembly_22c0dde4_joint_jointbody
- removed link AP-Assembly_8fe40f7e
- removed link AP-Assembly_8fe40f7e_joint_jointbody
- removed link AP-Assembly_a3d92f10
- removed link AP-Assembly_a3d92f10_joint_jointbody
- removed link CarpalsAssembly_a3f178b9
- removed link CarpalsAssembly_a3f178b9_joint_jointbody
- removed link FingerTipAssembly_28a83376
- removed link FingerTipAssembly_28a83376_joint_jointbody
- removed link FingerTipAssembly_a13adc36
- removed link FingerTipAssembly_a13adc36_joint_jointbody
- removed link FingerTipAssembly_bc7e70d7
- removed link FingerTipAssembly_bc7e70d7_joint_jointbody
- removed link FingerTipAssembly_cc9cd17e
- removed link FingerTipAssembly_cc9cd17e_joint_jointbody
- removed link I-PP-Assembly_32ddceb4
- removed link I-PP-Assembly_32ddceb4_joint_jointbody
- removed link M-PP-Assembly_8bc6ddb7
- removed link M-PP-Assembly_8bc6ddb7_joint_jointbody
- removed link M-PP-Assembly_c004e538
- removed link M-PP-Assembly_c004e538_joint_jointbody
- removed link P-PP-Assembly_4e31112a
- removed link P-PP-Assembly_4e31112a_joint_jointbody
- removed link P-PP-Assembly_c1041f9e
- removed link P-PP-Assembly_c1041f9e_joint_jointbody
- removed link T-AP-Assembly_b68d2db9
- removed link T-AP-Assembly_b68d2db9_joint_jointbody
- removed link T-TP-Assembly_8f310e51
- removed link T-TP-Assembly_8f310e51_joint_jointbody
- removed link ThumbTipAssembly_da16f050
- removed link ThumbTipAssembly_da16f050_joint_jointbody
- removed link TowerAssembly_8e26df17
- removed link root2TowerAssembly_8e26df17_fixed_jointbody
- added link index_abd_jointbody, mass 0.001
- added link index_fingertip, mass 0.0
- added link index_mp, mass 0.018229214728618118; visual mesh filename=package://viz/models/orca_test/urdf/converted_FingerTipAsse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
- added link index_mp2index_fingertip_fixed_jointbody, mass 0.001
- added link index_pp, mass 0.018700586463984262; visual mesh filename=package://viz/models/orca_test/urdf/converted_I-PP-Assembly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
- added link index_pp2mp_jointbody, mass 0.001
- added link index_um, mass 0.006625913032045117; visual mesh filename=package://viz/models/orca_test/urdf/converted_AP-Assembly.s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
- added link middle_abd_jointbody, mass 0.001
- added link middle_fingertip, mass 0.0
- added link middle_mp, mass 0.018229214728618118; visual mesh filename=package://viz/models/orca_test/urdf/converted_FingerTipAsse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
- added link middle_mp2middle_fingertip_fixed_jointbody, mass 0.001
- added link middle_pp, mass 0.023556963904505242; visual mesh filename=package://viz/models/orca_test/urdf/converted_M-PP-Assembly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
- added link middle_pp2mp_jointbody, mass 0.001
- added link middle_um, mass 0.006625913032045117; visual mesh filename=package://viz/models/orca_test/urdf/converted_AP-Assembly.s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
- added link palm, mass 0.2126860092978223; visual mesh filename=package://viz/models/orca_test/urdf/converted_CarpalsAssemb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
- added link pinky_abd_jointbody, mass 0.001
- added link pinky_fingertip, mass 0.0
- added link pinky_mp, mass 0.018229214728618118; visual mesh filename=package://viz/models/orca_test/urdf/converted_FingerTipAsse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
- added link pinky_mp2pinky_fingertip_fixed_jointbody, mass 0.001
- added link pinky_pp, mass 0.015497848277221124; visual mesh filename=package://viz/models/orca_test/urdf/converted_P-PP-Assembly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
- added link pinky_pp2mp_jointbody, mass 0.001
- added link pinky_um, mass 0.006625913032045117; visual mesh filename=package://viz/models/orca_test/urdf/converted_AP-Assembly.s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
- added link ring_abd_jointbody, mass 0.001
- added link ring_fingertip, mass 0.0
- added link ring_mp, mass 0.018229214728618118; visual mesh filename=package://viz/models/orca_test/urdf/converted_FingerTipAsse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
- added link ring_mp2ring_fingertip_fixed_jointbody, mass 0.001
- added link ring_pp, mass 0.023556963904505242; visual mesh filename=package://viz/models/orca_test/urdf/converted_M-PP-Assembly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
- added link ring_pp2mp_jointbody, mass 0.001
- added link ring_um, mass 0.006625913032045117; visual mesh filename=package://viz/models/orca_test/urdf/converted_AP-Assembly.s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
- added link root2index_pp_jointbody, mass 0.001
- added link root2middle_pp_jointbody, mass 0.001
- added link root2pinky_pp_jointbody, mass 0.001
- added link root2ring_pp_jointbody, mass 0.001
- added link root2thumb_base_jointbody, mass 0.001
- added link root2tower_fixed_jointbody, mass 0.001
- added link thumb_base, mass 0.0074875144010899545; visual mesh filename=package://viz/models/orca_test/urdf/converted_T-TP-Assembly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
- added link thumb_base2pp_jointbody, mass 0.001
- added link thumb_dp, mass 0.01818889883021656; visual mesh filename=package://viz/models/orca_test/urdf/converted_ThumbTipAssem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
- added link thumb_dp2thumb_fingertip_fixed_jointbody, mass 0.001
- added link thumb_fingertip, mass 0.0
- added link thumb_mp, mass 0.015497848277221124; visual mesh filename=package://viz/models/orca_test/urdf/converted_P-PP-Assembly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
- added link thumb_mp2dp_jointbody, mass 0.001
- added link thumb_pp, mass 0.01402737042708516; visual mesh filename=package://viz/models/orca_test/urdf/converted_T-AP-Assembly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
- added link thumb_pp2mp_jointbody, mass 0.001
- added link tower, mass 2.9399146871191753; visual mesh filename=package://viz/models/orca_test/urdf/converted_TowerAssembly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
- added link tower2root_jointbody, mass 0.001
Joints:
- removed joint AP-Assembly_0c2e1cd6_joint
- removed joint AP-Assembly_0c2e1cd6_joint_offset
- removed joint AP-Assembly_22c0dde4_joint
- removed joint AP-Assembly_22c0dde4_joint_offset
- removed joint AP-Assembly_8fe40f7e_joint
- removed joint AP-Assembly_8fe40f7e_joint_offset
- removed joint AP-Assembly_a3d92f10_joint
- removed joint AP-Assembly_a3d92f10_joint_offset
- removed joint CarpalsAssembly_a3f178b9_joint
- removed joint CarpalsAssembly_a3f178b9_joint_offset
- removed joint FingerTipAssembly_28a83376_joint
- removed joint FingerTipAssembly_28a83376_joint_offset
- removed joint FingerTipAssembly_a13adc36_joint
- removed joint FingerTipAssembly_a13adc36_joint_offset
- removed joint FingerTipAssembly_bc7e70d7_joint
- removed joint FingerTipAssembly_bc7e70d7_joint_offset
- removed joint FingerTipAssembly_cc9cd17e_joint
- removed joint FingerTipAssembly_cc9cd17e_joint_offset
- removed joint I-PP-Assembly_32ddceb4_joint
- removed joint I-PP-Assembly_32ddceb4_joint_offset
- removed joint M-PP-Assembly_8bc6ddb7_joint
- removed joint M-PP-Assembly_8bc6ddb7_joint_offset
- removed joint M-PP-Assembly_c004e538_joint
- removed joint M-PP-Assembly_c004e538_joint_offset
- removed joint P-PP-Assembly_4e31112a_joint
- removed joint P-PP-Assembly_4e31112a_joint_offset
- removed joint P-PP-Assembly_c1041f9e_joint
- removed joint P-PP-Assembly_c1041f9e_joint_offset
- removed joint T-AP-Assembly_b68d2db9_joint
- removed joint T-AP-Assembly_b68d2db9_joint_offset
- removed joint T-TP-Assembly_8f310e51_joint
- removed joint T-TP-Assembly_8f310e51_joint_offset
- removed joint ThumbTipAssembly_da16f050_joint
- removed joint ThumbTipAssembly_da16f050_joint_offset
- removed joint root2TowerAssembly_8e26df17_fixed
- removed joint root2TowerAssembly_8e26df17_fixed_offset
- added joint index_abd: type revolute, parent palm, child index_abd_jointbody, origin xyz=-0.02409178493002779 0.0019042822195537534 0.025160679302658893 rpy=1.608102038715379 1.1529632074851635 -0.051848338904223135, axis 4.163336342344337e-17 9.992007221626409e-16 -1.0000000000000013, limit lower=-0.5235987755982988 upper=0.5235987755982988 effort=100 velocity=100
- added joint index_abd_offset: type fixed, parent index_abd_jointbody, child index_um, origin xyz=-0.020000000000000052 2.3852447794681098e-18 -4.336808689942018e-19 rpy=0.0 0.0 0.0
- added joint index_mp2index_fingertip_fixed: type fixed, parent index_mp, child index_mp2index_fingertip_fixed_jointbody, origin xyz=-0.009 0.0 0.04 rpy=0.0 0.0 0.0
- added joint index_mp2index_fingertip_fixed_offset: type fixed, parent index_mp2index_fingertip_fixed_jointbody, child index_fingertip, origin xyz=-0.0 -0.0 -0.0 rpy=0.0 0.0 0.0
- added joint index_pp2mp: type revolute, parent index_pp, child index_pp2mp_jointbody, origin xyz=0.0004999999999839601 6.589248156966668e-17 0.038 rpy=0.0 0.0 1.1102230246251565e-16, axis -1.1102230246251565e-15 -0.9999999999999998 -8.326672684688674e-17, limit lower=-0.3490658503988659 upper=2.2689280275926285 effort=100 velocity=100
- added joint index_pp2mp_offset: type fixed, parent index_pp2mp_jointbody, child index_mp, origin xyz=4.506562989359519e-18 -5.895358766575946e-17 -6.487401240321147e-17 rpy=0.0 0.0 0.0
- added joint middle_abd: type revolute, parent palm, child middle_abd_jointbody, origin xyz=4.881579836291013e-18 -8.567697285510997e-18 0.03 rpy=1.5707963267948966 1.5707963267948966 0.0, axis -9.645057161491277e-31 -1.6653345369377348e-16 -0.9999999999999998, limit lower=-0.5235987755982988 upper=0.5235987755982988 effort=100 velocity=100
- added joint middle_abd_offset: type fixed, parent middle_abd_jointbody, child middle_um, origin xyz=-0.019999999999999987 -3.771356811665857e-18 1.701695755040975e-18 rpy=0.0 0.0 0.0
- added joint middle_mp2middle_fingertip_fixed: type fixed, parent middle_mp, child middle_mp2middle_fingertip_fixed_jointbody, origin xyz=-0.009 0.0 0.04 rpy=0.0 0.0 0.0
- added joint middle_mp2middle_fingertip_fixed_offset: type fixed, parent middle_mp2middle_fingertip_fixed_jointbody, child middle_fingertip, origin xyz=-0.0 -0.0 -0.0 rpy=0.0 0.0 0.0
- added joint middle_pp2mp: type revolute, parent middle_pp, child middle_pp2mp_jointbody, origin xyz=0.0004999999999727624 -3.4694469519535125e-18 0.04600000000000015 rpy=0.0 0.0 0.0, axis 1.1102230246251565e-16 -1.0000000000000004 -2.7755575615628914e-17, limit lower=-0.3490658503988659 upper=2.2689280275926285 effort=100 velocity=100
- added joint middle_pp2mp_offset: type fixed, parent middle_pp2mp_jointbody, child middle_mp, origin xyz=-5.421010862428354e-19 -1.0168910106364605e-31 -8.326672684688675e-17 rpy=0.0 0.0 0.0
- added joint pinky_abd: type revolute, parent palm, child pinky_abd_jointbody, origin xyz=0.04258768282792981 0.004991925321003577 0.007247738795820427 rpy=-1.4969430651841689 0.8614853700810636 -2.883730096597108, axis 1.942890293094024e-16 -5.551115123125783e-16 -0.9999999999999997, limit lower=-0.5235987755982988 upper=0.5235987755982988 effort=100 velocity=100
- added joint pinky_abd_offset: type fixed, parent pinky_abd_jointbody, child pinky_um, origin xyz=-0.020000000000000014 -2.42861286636753e-17 -6.071532165918825e-18 rpy=0.0 0.0 0.0
- added joint pinky_mp2pinky_fingertip_fixed: type fixed, parent pinky_mp, child pinky_mp2pinky_fingertip_fixed_jointbody, origin xyz=-0.009 0.0 0.04 rpy=0.0 0.0 0.0
- added joint pinky_mp2pinky_fingertip_fixed_offset: type fixed, parent pinky_mp2pinky_fingertip_fixed_jointbody, child pinky_fingertip, origin xyz=-0.0 -0.0 -0.0 rpy=0.0 0.0 0.0
- added joint pinky_pp2mp: type revolute, parent pinky_pp, child pinky_pp2mp_jointbody, origin xyz=0.0004999999999844908 -2.39390297194962e-18 0.032999999999999946 rpy=-1.1102230246251565e-16 0.0 -1.1102230246251565e-16, axis -2.7755575615628914e-16 -1.0000000000000007 -2.498001805406602e-16, limit lower=-0.3490658503988659 upper=2.2689280275926285 effort=100 velocity=100
- added joint pinky_pp2mp_offset: type fixed, parent pinky_pp2mp_jointbody, child pinky_mp, origin xyz=4.630531374131085e-18 3.7088372491485756e-17 3.145406773126967e-17 rpy=0.0 0.0 0.0
- added joint ring_abd: type revolute, parent palm, child ring_abd_jointbody, origin xyz=0.02151626244325177 0.001539966070889325 0.02082193721565796 rpy=-1.5359724334240115 1.3083608795701225 -3.054411807001147, axis 2.0816681711721685e-16 -1.1102230246251565e-16 -0.9999999999999998, limit lower=-0.5235987755982988 upper=0.5235987755982988 effort=100 velocity=100
- added joint ring_abd_offset: type fixed, parent ring_abd_jointbody, child ring_um, origin xyz=-0.020000000000000052 4.640385298237959e-17 -5.421010862427522e-18 rpy=0.0 0.0 0.0
- added joint ring_mp2ring_fingertip_fixed: type fixed, parent ring_mp, child ring_mp2ring_fingertip_fixed_jointbody, origin xyz=-0.009 0.0 0.04 rpy=0.0 0.0 0.0
- added joint ring_mp2ring_fingertip_fixed_offset: type fixed, parent ring_mp2ring_fingertip_fixed_jointbody, child ring_fingertip, origin xyz=-0.0 -0.0 -0.0 rpy=0.0 0.0 0.0
- added joint ring_pp2mp: type revolute, parent ring_pp, child ring_pp2mp_jointbody, origin xyz=0.0004999999999727536 -3.2334689427772335e-19 0.046000000000000194 rpy=5.551115123125783e-17 0.0 1.1102230246251565e-16, axis 0.0 -0.9999999999999998 -5.551115123125783e-17, limit lower=-0.3490658503988659 upper=2.2689280275926285 effort=100 velocity=100
- added joint ring_pp2mp_offset: type fixed, parent ring_pp2mp_jointbody, child ring_mp, origin xyz=6.5371804131346096e-18 1.5935858178068978e-17 -1.6822041242320552e-16 rpy=0.0 0.0 0.0
- added joint root2index_pp: type revolute, parent index_um, child root2index_pp_jointbody, origin xyz=-2.5541056475587942e-17 1.0557908552474885e-17 -8.628646044820514e-18 rpy=-7.850462293418875e-17 -1.5707963267948963 0.0, axis -1.1102230246251565e-15 -0.9999999999999998 -8.326672684688674e-17, limit lower=-0.3490658503988659 upper=1.9198621771937625 effort=100 velocity=100
- added joint root2index_pp_offset: type fixed, parent root2index_pp_jointbody, child index_pp, origin xyz=8.62864604482052e-18 -1.0557908552474884e-17 -2.5541056475587933e-17 rpy=0.0 0.0 0.0
- added joint root2middle_pp: type revolute, parent middle_um, child root2middle_pp_jointbody, origin xyz=-8.326672684688675e-17 1.0477058897466563e-31 9.860761315262648e-32 rpy=0.0 -1.5707963267948963 0.0, axis 1.1102230246251565e-16 -1.0000000000000004 -2.7755575615628914e-17, limit lower=-0.3490658503988659 upper=1.9198621771937625 effort=100 velocity=100
- added joint root2middle_pp_offset: type fixed, parent root2middle_pp_jointbody, child middle_pp, origin xyz=-8.011868568650901e-32 -1.0477058897466563e-31 -8.326672684688675e-17 rpy=0.0 0.0 0.0
- added joint root2pinky_pp: type revolute, parent pinky_um, child root2pinky_pp_jointbody, origin xyz=-9.80194474041885e-17 2.8970456895533516e-17 -1.0346526674750982e-18 rpy=7.850462293418872e-17 -1.5707963267948961 0.0, axis -1.6653345369377348e-16 -1.0000000000000004 -2.220446049250313e-16, limit lower=-0.3490658503988659 upper=1.9198621771937625 effort=100 velocity=100
- added joint root2pinky_pp_offset: type fixed, parent root2pinky_pp_jointbody, child pinky_pp, origin xyz=-3.4409772224679328e-18 -3.9175276362032155e-17 -1.0647123163719203e-16 rpy=0.0 0.0 0.0
- added joint root2ring_pp: type revolute, parent ring_um, child root2ring_pp_jointbody, origin xyz=5.000422469950927e-17 2.7821222532288604e-17 -6.247486316027035e-19 rpy=0.0 -1.5707963267948963 0.0, axis 0.0 -0.9999999999999998 -5.551115123125783e-17, limit lower=-0.3490658503988659 upper=1.9198621771937625 effort=100 velocity=100
- added joint root2ring_pp_offset: type fixed, parent root2ring_pp_jointbody, child ring_pp, origin xyz=6.247486316026924e-19 -2.7821222532288604e-17 5.000422469950927e-17 rpy=0.0 0.0 0.0
- added joint root2thumb_base: type revolute, parent palm, child root2thumb_base_jointbody, origin xyz=-0.026596228805379245 0.012467608905357173 -0.013731317517900202 rpy=-2.623243999248972 0.36429799059196055 -1.2778314442697774, axis -2.920774733183862e-12 3.3306690738754696e-16 1.0000000000000002, limit lower=-0.9250245035569946 upper=0.8377580409572782 effort=100 velocity=100
- added joint root2thumb_base_offset: type fixed, parent root2thumb_base_jointbody, child thumb_base, origin xyz=-0.016999999999975042 -6.852157730108388e-17 -2.7301511745791984e-14 rpy=0.0 0.0 0.0
- added joint root2tower_fixed: type fixed, parent root, child root2tower_fixed_jointbody, origin xyz=0.0 0.0 0.0 rpy=0.0 0.0 0.0
- added joint root2tower_fixed_offset: type fixed, parent root2tower_fixed_jointbody, child tower, origin xyz=-0.0 -0.0 -0.0 rpy=0.0 0.0 0.0
- added joint thumb_base2pp: type revolute, parent thumb_base, child thumb_base2pp_jointbody, origin xyz=-2.0816681711721685e-17 -0.006690243410563722 -0.00030669391648898483 rpy=1.9198621771937625 2.220446049250313e-16 -1.1102230246251565e-16, axis -1.1102230246251565e-16 0.34202014332566866 0.9396926207859075, limit lower=-0.7853981633974483 upper=0.7853981633974483 effort=100 velocity=100
- added joint thumb_base2pp_offset: type fixed, parent thumb_base2pp_jointbody, child thumb_pp, origin xyz=-0.03 -0.002 -0.0063916678614429154 rpy=0.0 0.0 0.0
- added joint thumb_dp2thumb_fingertip_fixed: type fixed, parent thumb_dp, child thumb_dp2thumb_fingertip_fixed_jointbody, origin xyz=0.0 0.0 0.03 rpy=0.0 0.0 0.0
- added joint thumb_dp2thumb_fingertip_fixed_offset: type fixed, parent thumb_dp2thumb_fingertip_fixed_jointbody, child thumb_fingertip, origin xyz=-0.0 -0.0 -0.0 rpy=0.0 0.0 0.0
- added joint thumb_mp2dp: type revolute, parent thumb_mp, child thumb_mp2dp_jointbody, origin xyz=0.0004999999999845258 1.960237527853792e-16 0.03299999999999989 rpy=-4.440892098500625e-16 -4.440892098500626e-16 -1.110223024625157e-15, axis -1.3877787807814457e-16 -1.0000000000000018 1.6653345369377348e-16, limit lower=-0.3490658503988659 upper=1.7453292519943295 effort=100 velocity=100
- added joint thumb_mp2dp_offset: type fixed, parent thumb_mp2dp_jointbody, child thumb_dp, origin xyz=0.0 0.0 -0.0 rpy=0.0 0.0 0.0
- added joint thumb_pp2mp: type revolute, parent thumb_pp, child thumb_pp2mp_jointbody, origin xyz=4.708523807784693e-17 1.513645907263937e-16 -4.2834101494079344e-17 rpy=-3.1415926535897927 1.5707963267948948 0.0, axis -1.27675647831893e-15 -0.9999999999999994 4.996003610813204e-16, limit lower=-0.3490658503988659 upper=2.007128639793479 effort=100 velocity=100
- added joint thumb_pp2mp_offset: type fixed, parent thumb_pp2mp_jointbody, child thumb_mp, origin xyz=0.0 0.0 0.0 rpy=0.0 0.0 0.0
- added joint tower2root: type revolute, parent tower, child tower2root_jointbody, origin xyz=0.04062890845062731 3.686287386450715e-18 0.10237107458169505 rpy=-6.123233995736781e-17 -4.440892098500626e-16 1.942890293094021e-16, axis -1.0000000000000009 -1.4791141972893971e-31 -1.0947644252537633e-46, limit lower=-1.0471975511965976 upper=1.0471975511965976 effort=100 velocity=100
- added joint tower2root_offset: type fixed, parent tower2root_jointbody, child palm, origin xyz=-0.002000000000000012 0.0014412498723578018 0.03871931353519552 rpy=0.0 0.0 0.0
