Commit message: paper: retargeter fix + name change

File: src/viz/models/orca_v1/urdf/orca_v1_nowrist.urdf (robot description, URDF)
Before this commit: robot converted_robot, 49 links, 48 joints
Links:
- removed link root2tower_fixed_jointbody
- removed link tower
- removed link tower2root_jointbody
- added link root2palm_fixed_jointbody, mass 0.001
- link index_mp: geometry visual mesh filename=package://viz/models/orca_v1/urdf/converted_FingerTipAssemb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
- link index_pp: geometry visual mesh filename=package://viz/models/orca_v1/urdf/converted_I-PP-Assembly.s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
- link index_um: geometry visual mesh filename=package://viz/models/orca_v1/urdf/converted_AP-Assembly.stl
- link middle_mp: geometry visual mesh filename=package://viz/models/orca_v1/urdf/converted_FingerTipAssemb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
- link middle_pp: geometry visual mesh filename=package://viz/models/orca_v1/urdf/converted_M-PP-Assembly.s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
- link middle_um: geometry visual mesh filename=package://viz/models/orca_v1/urdf/converted_AP-Assembly.stl
- link palm: geometry visual mesh filename=package://viz/models/orca_v1/urdf/converted_CarpalsAssembly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
- link pinky_mp: geometry visual mesh filename=package://viz/models/orca_v1/urdf/converted_FingerTipAssemb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
- link pinky_pp: geometry visual mesh filename=package://viz/models/orca_v1/urdf/converted_P-PP-Assembly.s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
- link pinky_um: geometry visual mesh filename=package://viz/models/orca_v1/urdf/converted_AP-Assembly.stl
- link ring_mp: geometry visual mesh filename=package://viz/models/orca_v1/urdf/converted_FingerTipAssemb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
- link ring_pp: geometry visual mesh filename=package://viz/models/orca_v1/urdf/converted_M-PP-Assembly.s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
- link ring_um: geometry visual mesh filename=package://viz/models/orca_v1/urdf/converted_AP-Assembly.stl
- link thumb_base: geometry visual mesh filename=package://viz/models/orca_v1/urdf/converted_T-TP-Assembly.s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
- link thumb_dp: geometry visual mesh filename=package://viz/models/orca_v1/urdf/converted_ThumbTipAssembl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
- link thumb_mp: geometry visual mesh filename=package://viz/models/orca_v1/urdf/converted_P-PP-Assembly.s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
- link thumb_pp: geometry visual mesh filename=package://viz/models/orca_v1/urdf/converted_T-AP-Assembly.s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
Joints:
- removed joint root2tower_fixed
- removed joint root2tower_fixed_offset
- removed joint tower2root
- removed joint tower2root_offset
- added joint root2palm_fixed: type fixed, parent root, child root2palm_fixed_jointbody, origin xyz=0.03862890845062728 0.0014412498723578074 0.14109038811689056 rpy=-6.123233995736781e-17 -4.440892098500626e-16 1.942890293094021e-16
- added joint root2palm_fixed_offset: type fixed, parent root2palm_fixed_jointbody, child palm, origin xyz=-0.0 -0.0 -0.0 rpy=0.0 0.0 0.0
